Commit message: Update xacro to include S model

File: phoxi_camera_ros2/urdf/M+_Motion_Cam-3D.xacro (robot description, xacro)
@@ -7,10 +7,4 @@
     prefix="${config['/**']['ros__parameters']['tf_prefix']}"
     phoxi_model="M+_Motion_Cam-3D"
-    x="0.0628"
-    y="-0.1728"
-    z="0.0326"
-    roll="${-pi / 2}"
-    pitch="0.0"
-    yaw="${-pi / 2}"
   />
 </robot>

File: phoxi_camera_ros2/urdf/phoxi.xacro (robot description, xacro)
@@ -1,10 +1,9 @@
 <?xml version="1.0"?>
 <robot name="phoxi" xmlns:xacro="http://ros.org/wiki/xacro">
-  <xacro:macro name="phoxi_macro" params="prefix phoxi_model x y z roll pitch yaw">
+  <xacro:macro name="phoxi_macro" params="prefix phoxi_model">
     <link name="${prefix}_base_link">
       <visual>
-        <origin rpy="0 0 0" xyz="0 0 0"/>
         <geometry>
-          <mesh scale="0.001 0.001 0.001" filename="package://phoxi_camera_ros2/meshes/${phoxi_model}.stl" />
+          <mesh filename="package://phoxi_camera_ros2/meshes/visual/${phoxi_model}.stl" />
         </geometry>
         <material name="dark">
@@ -12,7 +11,13 @@
         </material>
       </visual>
+      <collision>
+        <geometry>
+          <mesh filename="package://phoxi_camera_ros2/meshes/collision/${phoxi_model}.stl" />
+        </geometry>
+      </collision>
     </link>
+    <xacro:property name="pose" value="${xacro.load_yaml('$(find phoxi_camera_ros2)/param/camera_poses.yaml')[phoxi_model]}"/>
     <joint name="${prefix}_base_to_camera_joint" type="fixed">
-      <origin rpy="${roll} ${pitch} ${yaw}" xyz="${x} ${y} ${z}"/>
+      <origin rpy="${pose['rpy']}" xyz="${pose['xyz']}"/>
       <parent link="${prefix}_base_link"/>
       <child link="${prefix}_camera_link"/>
@@ -30,5 +35,5 @@
         <origin rpy="0 0 0" xyz="0 0 0"/>
         <geometry>
-          <mesh scale="0.001 0.001 0.001" filename="package://phoxi_camera_ros2/meshes/${phoxi_model}_FOV.stl" />
+          <mesh filename="package://phoxi_camera_ros2/meshes/visual/${phoxi_model}_FOV.stl" />
         </geometry>
         <material name="green">
