Commit message: Update urdf

File: phoxi_camera_ros2/urdf/phoxi.xacro (robot description, xacro)
@@ -26,5 +26,11 @@
       <origin rpy="0 0 0" xyz="0 0 0"/>
     </link>
-    <joint name="${prefix}_base_to_fov_joint" type="fixed">
+    <link name="${prefix}_camera_tool0"/>
+    <joint name="${prefix}_camera_tool0" type="fixed">
+      <origin xyz="0 0 ${pose['distance']}"/>
+      <parent link="${prefix}_camera_link"/>
+      <child link="${prefix}_camera_tool0"/>
+    </joint>
+    <!-- <joint name="${prefix}_base_to_fov_joint" type="fixed">
       <origin rpy="0 0 0" xyz="0 0 0"/>
       <parent link="${prefix}_base_link"/>
@@ -41,5 +47,5 @@
         </material>
       </visual>
-    </link>
+    </link> -->
   </xacro:macro>
 </robot>
